Commit message: Rtabmap integration

File: rae_description/urdf/rae.urdf.xacro (robot description, xacro)
@@ -273,5 +273,5 @@
   <link name="rae_imu_frame"/>
   <joint name="rae_imu_joint" type="fixed">
-    <origin xyz="0 0 0" rpy="0 0 0"/>
+    <origin xyz="0 0 0" rpy="0 3.14 -1.570796327"/>
     <parent link="base_link"/>
     <child link="rae_imu_frame"/>
